File: t41_2_main_board.kicad_pcb (KiCad board)
At the start: 2 copper layers, 100 x 100 mm, 46 parts, among them IC1 74HC125D, J1 Conn_02x08_Odd_Even, J10 SJ-3524-SMT, J11 B2B-XH-A_LF__SN_, J12 SJ-3524-SMT, J13 B3B-XH-A_LF__SN_, J15 B4B-XH-A_LF__SN_, J2 Conn_02x05_Odd_Even, J3 Conn_02x05_Odd_Even, J4 Conn_02x05_Odd_Even, J5 Conn_02x05_Odd_Even, J6 SJ-3524-SMT, J7 SJ-3524-SMT, J8 SJ-3524-SMT, J9 B3B-XH-A_LF__SN_, U1 Teensy4.1

Commit message: To fab.
Parts:
- added C14: 2.2nF, Capacitor_SMD:C_1206_3216Metric, F.Cu at (153.1, 135.1)
- added J14: B2B-XH-A_LF__SN_, digikey-footprints:PinHeader_1x2_P2.5mm_Drill1.1mm, F.Cu at (181.1, 70.5)
- added J16: B3B-XH-A_LF__SN_, digikey-footprints:PinHeader_1x3_P2.5mm_Drill1.1mm, F.Cu at (131.4, 134.6)
- added R1: 470, Resistor_SMD:R_1206_3216Metric, F.Cu at (157.0, 132.0)
Connections:
- C2 pad 1: Net-(U3-LROUT) -> Net-(C14-Pad2)
- J5 pad 7: unconnected-(J5-Pin_7-Pad7) -> /DISP_PWR
- J5 pad 8: unconnected-(J5-Pin_8-Pad8) -> /DISP_PWR
- U1 pad 33: unconnected-(U1-41_A17-Pad33) -> Net-(J4-Pin_6)
- U1 pad 36: Net-(J4-Pin_6) -> /SPDIF_OUT
- U3 pad 4: unconnected-(U3-AGND-Pad4) -> GND
- U3 pad 5: Net-(U3-A3V3) -> /3_3V_FIL
- U3 pad 7: Net-(U3-A3V3) -> /3_3V_FIL
Routing:
- net GND: track 515.9 -> 93.8 mm, vias 85 -> 128
- net /DISP_PWR: track 0.00 -> 113.2 mm
- net /3_3V_FIL: track 167.0 -> 207.4 mm, vias 1 -> 3
- net /SPDIF_OUT: track 0.00 -> 36.0 mm, vias 0 -> 1
- net Net-(C14-Pad2): track 0.00 -> 11.3 mm
- net Net-(U3-LROUT): track 24.4 -> 16.1 mm
- net Net-(U3-A3V3): track 7.16 -> 0.00 mm
- net /BCK: track 51.3 -> 55.9 mm
- net /5V_FIL: track 109.6 -> 113.1 mm
- net /MUTE: track 78.2 -> 81.1 mm
- net Net-(J4-Pin_6): track 47.7 -> 50.1 mm, vias 0 -> 1
- net Net-(C2-Pad2): track 52.0 -> 53.9 mm
- net /CS: track 34.4 -> 32.8 mm, vias 0 -> 2
- net /MOSI: track 12.8 -> 14.1 mm
- net /KEY2: track 49.0 -> 50.2 mm
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Other:
- board text added: "3.3V"
- board text added: "5V"
- board text added: "AUDIO OUT"
- board text added: "DISPLAY"
- board text added: "FILTER"
- board text added: "FINE TUNE"
- board text added: "KEY"
- board text added: "KF5N"
- board text added: "MATRIX"
- board text added: "MIC"
- board text added: "QSD"
- board text added: "QSE"
- board text added: "SPDIF"
- board text added: "SWITCH"
- board text added: "TUNE"
- board text added: "VOLUME"
